Commit message: navigation

File: tr3_description/urdf/arm/arm.gazebo.xacro (robot description, xacro)
@@ -15,4 +15,7 @@
 		<material>Gazebo/DarkGrey</material>
 	</gazebo>
+	<gazebo reference="link_a4">
+		<material>Gazebo/DarkGrey</material>
+	</gazebo>
 	<gazebo reference="link_g0">
 		<material>Gazebo/DarkGrey</material>
