Commit message: moveit integration

File: tr3_description/urdf/arm/arm.urdf.xacro (robot description, xacro)
@@ -12,4 +12,10 @@
 	<xacro:arm_link name="g1" mesh_name="xt-gp-b" origin_xyz="0 0 0" origin_rpy="1.5708 0 0" />
 	<xacro:arm_link name="g1_b" mesh_name="xt-gp-c" origin_xyz="0 0 0" origin_rpy="1.5708 0 0" />
+  <link name="link_g0_fixed">
+    <inertial>
+      <mass value="0.005"/>
+      <inertia ixx="0.001" iyy="0.001" izz="0.001" ixy="0" ixz="0" iyz="0" />
+    </inertial>
+  </link>
 	<joint name="a0" type="revolute">
 		<parent link="base_link"/>
@@ -60,4 +66,11 @@
     <dynamics damping="0.1" friction="0.1"/>
 	</joint>
+  <joint name="a4_fixed" type="fixed">
+		<parent link="link_g0"/>
+    <child link="link_g0_fixed"/>
+		<origin xyz="0 0 -0.235" rpy="0 0 0"/>
+    <axis xyz="0 0 1"/>
+    <dynamics damping="0.1" friction="0.1"/>
+  </joint>
 	<joint name="g0" type="prismatic">
 		<parent link="link_g0"/>

Commit message: joint direction

File: tr3_description/urdf/arm/arm.urdf.xacro (robot description, xacro)
@@ -22,5 +22,5 @@
 		<child link="link_a0"/>
 		<origin xyz="-0.1016 0.1229 0.459937" rpy="0 0 0"/>
-    <axis xyz="0 0 1"/>
+    <axis xyz="0 0 -1"/>
 		<limit effort="100.0" lower="-2" upper="2" velocity="0.20"/>
     <dynamics damping="0.1" friction="0.1"/>
@@ -30,5 +30,5 @@
 		<child link="link_a1"/>
 		<origin xyz="0.070 0.0000 0.076" rpy="0 0 0"/>
-    <axis xyz="1 0 0"/>
+    <axis xyz="-1 0 0"/>
 		<limit effort="100.0" lower="-15" upper="15" velocity="0.20"/>
     <dynamics damping="0.1" friction="0.1"/>

Commit message: moveit config

File: tr3_description/urdf/arm/arm.urdf.xacro (robot description, xacro)
@@ -23,5 +23,5 @@
 		<origin xyz="-0.1016 0.1229 0.459937" rpy="0 0 0"/>
     <axis xyz="0 0 -1"/>
-		<limit effort="100.0" lower="-2" upper="2" velocity="0.20"/>
+		<limit effort="100.0" lower="-10" upper="10" velocity="0.20"/>
     <dynamics damping="0.1" friction="0.1"/>
 	</joint>
@@ -31,5 +31,5 @@
 		<origin xyz="0.070 0.0000 0.076" rpy="0 0 0"/>
     <axis xyz="-1 0 0"/>
-		<limit effort="100.0" lower="-15" upper="15" velocity="0.20"/>
+		<limit effort="100.0" lower="-10" upper="10" velocity="0.20"/>
     <dynamics damping="0.1" friction="0.1"/>
 	</joint>
@@ -39,5 +39,4 @@
 		<origin xyz="0 0 -0.190" rpy="0 0 0"/>
     <axis xyz="1 0 0"/>
-		<limit effort="100.0" lower="-15" upper="15" velocity="0.20"/>
     <dynamics damping="0.1" friction="0.1"/>
 	</joint>
@@ -47,5 +46,5 @@
 		<origin xyz="0 0 0" rpy="-0.698132 0 0"/>
     <axis xyz="1 0 0"/>
-		<limit effort="100.0" lower="-15" upper="15" velocity="0.20"/>
+		<limit effort="100.0" lower="-10" upper="10" velocity="0.20"/>
     <dynamics damping="0.1" friction="0.1"/>
 	</joint>
@@ -55,5 +54,5 @@
 		<origin xyz="0.008 -0.3 0" rpy="0.698132 0 0"/>
     <axis xyz="1 0 0"/>
-		<limit effort="100.0" lower="-15" upper="15" velocity="0.20"/>
+		<limit effort="100.0" lower="-10" upper="10" velocity="0.20"/>
     <dynamics damping="0.1" friction="0.1"/>
 	</joint>
@@ -63,5 +62,5 @@
 		<origin xyz="0.067 0 -0.067" rpy="0 0 0"/>
     <axis xyz="0 0 1"/>
-		<limit effort="100.0" lower="-15" upper="15" velocity="0.20"/>
+		<limit effort="100.0" lower="-10" upper="10" velocity="0.20"/>
     <dynamics damping="0.1" friction="0.1"/>
 	</joint>

Commit message: tr3py and urdf

File: tr3_description/urdf/arm/arm.urdf.xacro (robot description, xacro)
@@ -23,5 +23,5 @@
 		<origin xyz="-0.1016 0.1229 0.459937" rpy="0 0 0"/>
     <axis xyz="0 0 -1"/>
-		<limit effort="100.0" lower="-2" upper="2" velocity="0.20"/>
+		<limit effort="100.0" lower="-2" upper="2" velocity="0.8"/>
     <dynamics damping="0.1" friction="0.1"/>
 	</joint>
@@ -31,5 +31,5 @@
 		<origin xyz="0.070 0.0000 0.076" rpy="0 0 0"/>
     <axis xyz="-1 0 0"/>
-		<limit effort="100.0" lower="-15" upper="15" velocity="0.20"/>
+		<limit effort="100.0" lower="-15" upper="15" velocity="0.80"/>
     <dynamics damping="0.1" friction="0.1"/>
 	</joint>
@@ -39,5 +39,5 @@
 		<origin xyz="0 0 -0.190" rpy="0 0 0"/>
     <axis xyz="1 0 0"/>
-		<limit effort="100.0" lower="-15" upper="15" velocity="0.20"/>
+		<limit effort="100.0" lower="-15" upper="15" velocity="0.80"/>
     <dynamics damping="0.1" friction="0.1"/>
 	</joint>
@@ -47,5 +47,5 @@
 		<origin xyz="0 0 0" rpy="-0.698132 0 0"/>
     <axis xyz="1 0 0"/>
-		<limit effort="100.0" lower="-15" upper="15" velocity="0.20"/>
+		<limit effort="100.0" lower="-15" upper="15" velocity="0.80"/>
     <dynamics damping="0.1" friction="0.1"/>
 	</joint>
@@ -55,5 +55,5 @@
 		<origin xyz="0.008 -0.3 0" rpy="0.698132 0 0"/>
     <axis xyz="1 0 0"/>
-		<limit effort="100.0" lower="-15" upper="15" velocity="0.20"/>
+		<limit effort="100.0" lower="-15" upper="15" velocity="0.80"/>
     <dynamics damping="0.1" friction="0.1"/>
 	</joint>
@@ -63,5 +63,5 @@
 		<origin xyz="0.067 0 -0.067" rpy="0 0 0"/>
     <axis xyz="0 0 1"/>
-		<limit effort="100.0" lower="-15" upper="15" velocity="0.20"/>
+		<limit effort="100.0" lower="-15" upper="15" velocity="0.80"/>
     <dynamics damping="0.1" friction="0.1"/>
 	</joint>

Commit message: tr3py and urdf

File: tr3_description/urdf/arm/arm.urdf.xacro (robot description, xacro)
@@ -23,5 +23,5 @@
 		<origin xyz="-0.1016 0.1229 0.459937" rpy="0 0 0"/>
     <axis xyz="0 0 -1"/>
-		<limit effort="100.0" lower="-10" upper="10" velocity="0.20"/>
+		<limit effort="100.0" lower="-10" upper="10" velocity="0.85"/>
     <dynamics damping="0.1" friction="0.1"/>
 	</joint>
@@ -31,5 +31,5 @@
 		<origin xyz="0.070 0.0000 0.076" rpy="0 0 0"/>
     <axis xyz="-1 0 0"/>
-		<limit effort="100.0" lower="-10" upper="10" velocity="0.20"/>
+		<limit effort="100.0" lower="-10" upper="10" velocity="0.85"/>
     <dynamics damping="0.1" friction="0.1"/>
 	</joint>
@@ -46,5 +46,5 @@
 		<origin xyz="0 0 0" rpy="-0.698132 0 0"/>
     <axis xyz="1 0 0"/>
-		<limit effort="100.0" lower="-10" upper="10" velocity="0.20"/>
+		<limit effort="100.0" lower="-10" upper="10" velocity="0.85"/>
     <dynamics damping="0.1" friction="0.1"/>
 	</joint>
@@ -54,5 +54,5 @@
 		<origin xyz="0.008 -0.3 0" rpy="0.698132 0 0"/>
     <axis xyz="1 0 0"/>
-		<limit effort="100.0" lower="-10" upper="10" velocity="0.20"/>
+		<limit effort="100.0" lower="-10" upper="10" velocity="0.85"/>
     <dynamics damping="0.1" friction="0.1"/>
 	</joint>
@@ -62,5 +62,5 @@
 		<origin xyz="0.067 0 -0.067" rpy="0 0 0"/>
     <axis xyz="0 0 1"/>
-		<limit effort="100.0" lower="-10" upper="10" velocity="0.20"/>
+		<limit effort="100.0" lower="-10" upper="10" velocity="0.85"/>
     <dynamics damping="0.1" friction="0.1"/>
 	</joint>

Commit message: navigation and urdf

File: tr3_description/urdf/arm/arm.urdf.xacro (robot description, xacro)
@@ -21,5 +21,5 @@
 		<parent link="base_link"/>
 		<child link="link_a0"/>
-		<origin xyz="-0.1016 0.1229 0.459937" rpy="0 0 0"/>
+		<origin xyz="0.1016 -0.1229 0.459937" rpy="0 0 3.1415"/>
     <axis xyz="0 0 -1"/>
 		<limit effort="100.0" lower="-10" upper="10" velocity="0.85"/>

File: tr3_description/urdf/base/base.urdf.xacro (robot description, xacro)
@@ -4,9 +4,9 @@
 	<xacro:include filename="$(find tr3_description)/urdf/base/base.transmission.xacro" />
 	<!-- wheel macros -->
-  <xacro:macro name="tr3_wheel" params="name *origin">
+  <xacro:macro name="tr3_wheel" params="name *origin *axis">
 		<joint name="${name}" type="continuous">
 			<parent link="base_link"/>
 			<child link="link_${name}"/>
-		  <axis xyz="0 1 0"/>
+			<xacro:insert_block name="axis" />
 			<limit effort="100.0" velocity="8.8"/>
 			<xacro:insert_block name="origin" />
@@ -41,8 +41,9 @@
         <mesh filename="package://tr3_description/meshes/stl/tr-bs-a.stl" scale="0.001 0.001 0.001"/>
 			</geometry>
-			<origin rpy="0 0 0" />
+			<origin rpy="0 0 3.1415" />
 		</collision>
 		<inertial>
-      	<mass value="0.5" />
+      	<mass value="1" />
+        <origin xyz="0 -0.300 0" />
 		    <inertia ixx="0.001" ixy="0.0" ixz="0.0" iyy="0.001" iyz="0.0" izz="0.001" />
 		</inertial>
@@ -54,11 +55,13 @@
         <color rgba="0.2 0.2 0.2 1"/>
       </material>
-			<origin rpy="0 0 0" />
+			<origin rpy="0 0 3.1415" />
 		</visual>
 	</link>
 	<xacro:tr3_wheel name="b0">
+    <axis xyz="0 -1 0"/>
 		<origin rpy="0 0 -1.5708" xyz="0.3281 0 0"/>
 	</xacro:tr3_wheel>
 	<xacro:tr3_wheel name="b1">
+    <axis xyz="0 1 0"/>
 		<origin rpy="0 0 1.5708" xyz="-0.3281 0 0"/>
 	</xacro:tr3_wheel>

File: tr3_description/urdf/head/head.gazebo.xacro (robot description, xacro)
@@ -6,5 +6,5 @@
 			<visualize>true</visualize>
 			<camera>
-				<pose>0 0 0 3.1415 -1.5708 -1.5708</pose>
+				<pose>0 0 0 0 -1.5708 1.5708</pose>
 				<horizontal_fov>1.0</horizontal_fov>
 				<image>

File: tr3_description/urdf/head/head.urdf.xacro (robot description, xacro)
@@ -67,10 +67,10 @@
 		<parent link="head_link"/>
 		<child link="camera_link"/>
-		<origin rpy="0 0 0" xyz="0.025 0.150 0.0"/>
+		<origin rpy="0 0 3.1415" xyz="-0.105 -0.145 0.085"/>
 	</joint>
 	<joint name="h0" type="revolute">
 		<parent link="base_link"/>
 		<child link="neck_link"/>
-		<origin xyz="0 0.3579 0.70325"/>
+		<origin rpy="0 0 3.1415" xyz="0 -0.3579 0.70325"/>
     <axis xyz="0 0 1"/>
 		<limit effort="100.0" lower="-15" upper="15" velocity="0.20"/>
@@ -81,5 +81,5 @@
 		<child link="head_link"/>
 		<origin xyz="0.067 -0.16617 0.24917" rpy="0 0 0"/>
-    <axis xyz="1 0 0"/>
+    <axis xyz="-1 0 0"/>
 		<limit effort="100.0" lower="-15" upper="15" velocity="0.20"/>
     <dynamics damping="0.1" friction="0.1"/>

Commit message: gazebo, navigation, and tr3_os optimizations

File: tr3_description/urdf/arm/arm.urdf.xacro (robot description, xacro)
@@ -21,5 +21,5 @@
 		<parent link="base_link"/>
 		<child link="link_a0"/>
-		<origin xyz="0.1016 -0.1229 0.459937" rpy="0 0 3.1415"/>
+		<origin xyz="-0.1229 -0.1016 0.459937" rpy="0 0 1.5708"/>
     <axis xyz="0 0 -1"/>
 		<limit effort="100.0" lower="-10" upper="10" velocity="0.85"/>

File: tr3_description/urdf/base/base.urdf.xacro (robot description, xacro)
@@ -9,5 +9,5 @@
 			<child link="link_${name}"/>
 			<xacro:insert_block name="axis" />
-			<limit effort="100.0" velocity="0.5"/>
+			<limit effort="100.0" velocity="1.0"/>
 			<xacro:insert_block name="origin" />
     	<dynamics damping="0.001" friction="0.1"/>
@@ -41,9 +41,9 @@
         <mesh filename="package://tr3_description/meshes/stl/tr-bs-a.stl" scale="0.001 0.001 0.001"/>
 			</geometry>
-			<origin rpy="0 0 3.1415" />
+			<origin rpy="0 0 1.5708" />
 		</collision>
 		<inertial>
-      	<mass value="1" />
-        <origin xyz="0 -0.300 0" />
+      	<mass value="10" />
+        <origin xyz="-0.300 0 0" />
 		    <inertia ixx="0.001" ixy="0.0" ixz="0.0" iyy="0.001" iyz="0.0" izz="0.001" />
 		</inertial>
@@ -55,5 +55,5 @@
         <color rgba="0.2 0.2 0.2 1"/>
       </material>
-			<origin rpy="0 0 3.1415" />
+			<origin rpy="0 0 1.5708" />
 		</visual>
 	</link>
@@ -145,5 +145,5 @@
     <parent link="base_link"/>
     <child link="link_b2"/>
-    <origin xyz="-0.147 -0.39975 -0.09635" rpy="0 3.1415 -1.5708"/>
+    <origin xyz="-0.39975 -0.147 -0.09635" rpy="0 3.1415 3.1415"/>
     <axis xyz="0 0 1"/>
     <dynamics damping="0.1" friction="0.1"/>
@@ -159,5 +159,5 @@
     <parent link="base_link"/>
     <child link="link_b4"/>
-    <origin xyz="0.147 -0.39975 -0.09635" rpy="0 3.1415 -1.5708"/>
+    <origin xyz="-0.39975 0.147 -0.09635" rpy="0 3.1415 3.1415"/>
     <axis xyz="0 0 1"/>
     <dynamics damping="0.1" friction="0.1"/>
@@ -172,5 +172,5 @@
   <joint name="rplidar_joint" type="fixed">
     <axis xyz="0 0 1" />
-    <origin xyz="0 0.11 0" rpy="0 0 0" />
+    <origin xyz="0.11 0 0" rpy="0 0 -1.5708" />
     <parent link="base_link" />
     <child link="laser" />
@@ -179,10 +179,10 @@
   </link>
 	<xacro:tr3_wheel name="b0">
-    <axis xyz="0 -1 0"/>
-		<origin rpy="0 0 -1.5708" xyz="0.3281 0 0"/>
+    <axis xyz="0 1 0"/>
+		<origin rpy="0 0 0" xyz="0 0.3281 0"/>
 	</xacro:tr3_wheel>
 	<xacro:tr3_wheel name="b1">
-    <axis xyz="0 1 0"/>
-		<origin rpy="0 0 1.5708" xyz="-0.3281 0 0"/>
+    <axis xyz="0 -1 0"/>
+		<origin rpy="0 0 3.1415" xyz="0 -0.3281 0"/>
 	</xacro:tr3_wheel>
 </robot>

File: tr3_description/urdf/head/head.urdf.xacro (robot description, xacro)
@@ -72,5 +72,5 @@
 		<parent link="base_link"/>
 		<child link="neck_link"/>
-		<origin rpy="0 0 3.1415" xyz="0 -0.3579 0.70325"/>
+		<origin xyz="-0.3579 0 0.70325" rpy="0 0 1.5708" />
     <axis xyz="0 0 1"/>
 		<limit effort="100.0" lower="-15" upper="15" velocity="0.20"/>

Commit message: navigation tuning, gazebo tuning, tr3_os map + lidar display in render

File: tr3_description/urdf/arm/arm.urdf.xacro (robot description, xacro)
@@ -9,5 +9,5 @@
   <xacro:arm_link name="a3" mesh_name="xt-sm-c" origin_xyz="0.008 -0.3 0" origin_rpy="0 -1.5708 1.5708" />
   <xacro:arm_link name="a4" mesh_name="xt-sm-b" origin_xyz="0.067 0 -0.067" origin_rpy="1.5708 0 -1.5708" />
-  <xacro:arm_link name="g0" mesh_name="xt-gp-a" origin_xyz="0 0 0" origin_rpy="1.5708 0 1.5708" />
+  <xacro:arm_link name="g0" mesh_name="xt-gp-a" origin_xyz="0 0 -0.120" origin_rpy="3.1415 0 1.5708" />
 	<xacro:arm_link name="g1" mesh_name="xt-gp-b" origin_xyz="0 0 0" origin_rpy="1.5708 0 0" />
 	<xacro:arm_link name="g1_b" mesh_name="xt-gp-c" origin_xyz="0 0 0" origin_rpy="1.5708 0 0" />

File: tr3_description/urdf/base/base.gazebo.xacro (robot description, xacro)
@@ -37,6 +37,5 @@
 	<gazebo reference="link_b0">
 		<material>Gazebo/DarkGrey</material>
-    <mu1 value="100000.0"/>
-    <mu2 value="100000.0"/>
+    <turnGravityOff>false</turnGravityOff>
 		<collision>
       <surface>
@@ -60,6 +59,5 @@
 	<gazebo reference="link_b1">
 		<material>Gazebo/DarkGrey</material>
-    <mu1 value="100000.0"/>
-    <mu2 value="100000.0"/>
+    <turnGravityOff>false</turnGravityOff>
 		<collision>
       <surface>
@@ -86,5 +84,5 @@
     <kp value="10000000.0"/>
     <kd value="1.0"/>
-    <fdir1 value="1 0 0"/>
+    <fdir1 value="0 0 1"/>
   	<material>Gazebo/DarkGrey</material>
     <turnGravityOff>false</turnGravityOff>
@@ -104,5 +102,5 @@
     <kp value="10000000.0"/>
     <kd value="1.0"/>
-    <fdir1 value="1 0 0"/>
+    <fdir1 value="0 0 1"/>
   	<material>Gazebo/DarkGrey</material>
     <turnGravityOff>false</turnGravityOff>

File: tr3_description/urdf/base/base.urdf.xacro (robot description, xacro)
@@ -21,7 +21,7 @@
 			</collision>
 			<inertial>
-      	<mass value="0.01" />
-		    <inertia ixx="0.001" ixy="0.0" ixz="0.0" iyy="0.001" iyz="0.0" izz="0.001" />
-				</inertial>
+      	<mass value="10" />
+		    <inertia ixx="0.01" ixy="0.0" ixz="0.0" iyy="0.01" iyz="0.0" izz="0.01" />
+			</inertial>
 			<visual>
 				<geometry>
@@ -45,5 +45,5 @@
 		<inertial>
       	<mass value="10" />
-        <origin xyz="-0.300 0 0" />
+        <origin xyz="-0.300 0 0.100" />
 		    <inertia ixx="0.001" ixy="0.0" ixz="0.0" iyy="0.001" iyz="0.0" izz="0.001" />
 		</inertial>
@@ -66,6 +66,6 @@
     </collision>
     <inertial>
-        <mass value="0.01" />
-        <inertia ixx="0.001" ixy="0.0" ixz="0.0" iyy="0.001" iyz="0.0" izz="0.001" />
+        <mass value="0.1" />
+        <inertia ixx="0.0001" ixy="0.0" ixz="0.0" iyy="0.0001" iyz="0.0" izz="0.0001" />
     </inertial>
     <visual>
@@ -87,6 +87,6 @@
     </collision>
     <inertial>
-        <mass value="0.01" />
-        <inertia ixx="0.001" ixy="0.0" ixz="0.0" iyy="0.001" iyz="0.0" izz="0.001" />
+        <mass value="0.1" />
+        <inertia ixx="0.0001" ixy="0.0" ixz="0.0" iyy="0.0001" iyz="0.0" izz="0.0001" />
     </inertial>
     <visual>
@@ -108,6 +108,6 @@
     </collision>
     <inertial>
-        <mass value="0.01" />
-        <inertia ixx="0.001" ixy="0.0" ixz="0.0" iyy="0.001" iyz="0.0" izz="0.001" />
+        <mass value="0.1" />
+        <inertia ixx="0.0001" ixy="0.0" ixz="0.0" iyy="0.0001" iyz="0.0" izz="0.0001" />
     </inertial>
     <visual>
@@ -129,6 +129,6 @@
     </collision>
     <inertial>
-        <mass value="0.01" />
-        <inertia ixx="0.001" ixy="0.0" ixz="0.0" iyy="0.001" iyz="0.0" izz="0.001" />
+        <mass value="0.1" />
+        <inertia ixx="0.0001" ixy="0.0" ixz="0.0" iyy="0.0001" iyz="0.0" izz="0.0001" />
     </inertial>
     <visual>
@@ -142,12 +142,12 @@
     </visual>
   </link>
-  <joint name="b2" type="continuous">
+  <joint name="b2" type="fixed">
     <parent link="base_link"/>
     <child link="link_b2"/>
-    <origin xyz="-0.39975 -0.147 -0.09635" rpy="0 3.1415 3.1415"/>
+    <origin xyz="-0.39975 -0.147 -0.097" rpy="0 3.1415 3.1415"/>
     <axis xyz="0 0 1"/>
     <dynamics damping="0.1" friction="0.1"/>
   </joint>
-  <joint name="b3" type="continuous">
+  <joint name="b3" type="fixed">
     <parent link="link_b2"/>
     <child link="link_b3"/>
@@ -156,12 +156,12 @@
     <dynamics damping="0.1" friction="0.1"/>
   </joint>
-  <joint name="b4" type="continuous">
+  <joint name="b4" type="fixed">
     <parent link="base_link"/>
     <child link="link_b4"/>
-    <origin xyz="-0.39975 0.147 -0.09635" rpy="0 3.1415 3.1415"/>
+    <origin xyz="-0.39975 0.147 -0.097" rpy="0 3.1415 3.1415"/>
     <axis xyz="0 0 1"/>
     <dynamics damping="0.1" friction="0.1"/>
   </joint>
-  <joint name="b5" type="continuous">
+  <joint name="b5" type="fixed">
     <parent link="link_b4"/>
     <child link="link_b5"/>

Commit message: arm geometry changes, joint limits for moveit optimization

File: tr3_description/urdf/arm/arm.urdf.xacro (robot description, xacro)
@@ -21,7 +21,7 @@
 		<parent link="base_link"/>
 		<child link="link_a0"/>
-		<origin xyz="-0.1229 -0.1016 0.459937" rpy="0 0 1.5708"/>
+		<origin xyz="-0.1229 -0.1016 0.459937" rpy="0 0 0"/>
     <axis xyz="0 0 -1"/>
-		<limit effort="100.0" lower="-10" upper="10" velocity="0.85"/>
+		<limit effort="100.0" lower="-0.85" upper="2.00" velocity="0.85"/>
     <dynamics damping="0.1" friction="0.1"/>
 	</joint>
@@ -29,7 +29,7 @@
 		<parent link="link_a0"/>
 		<child link="link_a1"/>
-		<origin xyz="0.070 0.0000 0.076" rpy="0 0 0"/>
+		<origin xyz="0.133 0.063 0.076" rpy="0 0 1.5708"/>
     <axis xyz="-1 0 0"/>
-		<limit effort="100.0" lower="-10" upper="10" velocity="0.85"/>
+		<limit effort="100.0" lower="-0.48" upper="3.33" velocity="0.85"/>
     <dynamics damping="0.1" friction="0.1"/>
 	</joint>
@@ -46,5 +46,5 @@
 		<origin xyz="0 0 0" rpy="-0.698132 0 0"/>
     <axis xyz="1 0 0"/>
-		<limit effort="100.0" lower="-10" upper="10" velocity="0.85"/>
+		<limit effort="100.0" lower="-0.37" upper="4.60" velocity="0.85"/>
     <dynamics damping="0.1" friction="0.1"/>
 	</joint>
@@ -54,5 +54,5 @@
 		<origin xyz="0.008 -0.3 0" rpy="0.698132 0 0"/>
     <axis xyz="1 0 0"/>
-		<limit effort="100.0" lower="-10" upper="10" velocity="0.85"/>
+		<limit effort="100.0" lower="-4.71" upper="0.48" velocity="0.85"/>
     <dynamics damping="0.1" friction="0.1"/>
 	</joint>
@@ -62,5 +62,5 @@
 		<origin xyz="0.067 0 -0.067" rpy="0 0 0"/>
     <axis xyz="0 0 1"/>
-		<limit effort="100.0" lower="-10" upper="10" velocity="0.85"/>
+		<limit effort="100.0" lower="-6.28" upper="6.28" velocity="0.85"/>
     <dynamics damping="0.1" friction="0.1"/>
 	</joint>

Commit message: fixing joint direction

File: tr3_description/urdf/arm/arm.urdf.xacro (robot description, xacro)
@@ -53,6 +53,7 @@
 		<child link="link_a4"/>
 		<origin xyz="0.008 -0.3 0" rpy="0.698132 0 0"/>
-    <axis xyz="1 0 0"/>
-		<limit effort="100.0" lower="-4.71" upper="0.48" velocity="0.85"/>
+    <axis xyz="-1 0 0"/>
+    <!--limit effort="100.0" lower="-0.48" upper="4.71" velocity="0.85"/-->
+    <limit effort="100.0" lower="-6.28" upper="6.28" velocity="0.85"/>
     <dynamics damping="0.1" friction="0.1"/>
 	</joint>

Commit message: ik, gui fixing joint rotation

File: tr3_description/urdf/arm/arm.urdf.xacro (robot description, xacro)
@@ -54,6 +54,5 @@
 		<origin xyz="0.008 -0.3 0" rpy="0.698132 0 0"/>
     <axis xyz="-1 0 0"/>
-    <!--limit effort="100.0" lower="-0.48" upper="4.71" velocity="0.85"/-->
-    <limit effort="100.0" lower="-6.28" upper="6.28" velocity="0.85"/>
+    <limit effort="100.0" lower="-0.48" upper="4.71" velocity="0.85"/>
     <dynamics damping="0.1" friction="0.1"/>
 	</joint>
