Commit message: sim lidar and tr os minimap

File: tr3_description/urdf/base/base.gazebo.xacro (robot description, xacro)
@@ -22,4 +22,35 @@
 		</collision>
 	</gazebo>
+  <gazebo reference="laser">
+    <sensor type="gpu_ray" name="head_rplidar_sensor">
+      <pose>0 0 0.06 0 0 0</pose>
+      <visualize>false</visualize>
+      <update_rate>40</update_rate>
+      <ray>
+        <scan>
+          <horizontal>
+            <samples>720</samples>
+            <resolution>1</resolution>
+            <min_angle>0.26</min_angle>
+            <max_angle>2.88</max_angle>
+          </horizontal>
+        </scan>
+        <range>
+          <min>0.2</min>
+          <max>12.0</max>
+          <resolution>0.01</resolution>
+        </range>
+        <noise>
+          <type>gaussian</type>
+          <mean>0.0</mean>
+          <stddev>0.01</stddev>
+        </noise>
+      </ray>
+      <plugin name="gazebo_ros_head_rplidar_controller" filename="libgazebo_ros_gpu_laser.so">
+        <topicName>/tr3/lidar</topicName>
+        <frameName>laser</frameName>
+      </plugin>
+    </sensor>
+  </gazebo>
 	<gazebo reference="base_link">
 		<material>Gazebo/DarkGrey</material>

File: tr3_description/urdf/base/base.urdf.xacro (robot description, xacro)
@@ -58,4 +58,12 @@
 		</visual>
 	</link>
+  <joint name="rplidar_joint" type="fixed">
+    <axis xyz="0 0 1" />
+    <origin xyz="0 0.11 0" rpy="0 0 0" />
+    <parent link="base_link" />
+    <child link="laser" />
+  </joint>
+  <link name="laser">
+  </link>
 	<xacro:tr3_wheel name="b0">
     <axis xyz="0 -1 0"/>

Commit message: added SLAM

File: tr3_description/urdf/base/base.gazebo.xacro (robot description, xacro)
@@ -83,3 +83,9 @@
 		<material>Gazebo/DarkGrey</material>
 	</gazebo>
+	<gazebo reference="link_b4">
+		<material>Gazebo/DarkGrey</material>
+	</gazebo>
+	<gazebo reference="link_b5">
+		<material>Gazebo/DarkGrey</material>
+	</gazebo>
 </robot>

File: tr3_description/urdf/base/base.urdf.xacro (robot description, xacro)
@@ -58,4 +58,116 @@
 		</visual>
 	</link>
+  <link name="link_b2">
+    <collision>
+      <geometry>
+        <mesh filename="package://tr3_description/meshes/stl/tr-bs-b.stl" scale="0.001 0.001 0.001"/>
+      </geometry>
+      <origin rpy="0 0 1.5708" />
+    </collision>
+    <inertial>
+        <mass value="0.01" />
+        <inertia ixx="0.001" ixy="0.0" ixz="0.0" iyy="0.001" iyz="0.0" izz="0.001" />
+    </inertial>
+    <visual>
+      <geometry>
+        <mesh filename="package://tr3_description/meshes/stl/tr-bs-b.stl" scale="0.001 0.001 0.001"/>
+      </geometry>
+      <material name="slate_gray">
+        <color rgba="0.2 0.2 0.2 1"/>
+      </material>
+      <origin rpy="0 0 1.5708" />
+    </visual>
+  </link>
+  <link name="link_b3">
+    <collision>
+      <geometry>
+        <mesh filename="package://tr3_description/meshes/stl/tr-bs-c.stl" scale="0.001 0.001 0.001"/>
+      </geometry>
+      <origin rpy="0 0 1.5708" />
+    </collision>
+    <inertial>
+        <mass value="0.01" />
+        <inertia ixx="0.001" ixy="0.0" ixz="0.0" iyy="0.001" iyz="0.0" izz="0.001" />
+    </inertial>
+    <visual>
+      <geometry>
+        <mesh filename="package://tr3_description/meshes/stl/tr-bs-c.stl" scale="0.001 0.001 0.001"/>
+      </geometry>
+      <material name="slate_gray">
+        <color rgba="0.2 0.2 0.2 1"/>
+      </material>
+      <origin rpy="0 0 1.5708" />
+    </visual>
+  </link>
+  <link name="link_b4">
+    <collision>
+      <geometry>
+        <mesh filename="package://tr3_description/meshes/stl/tr-bs-b.stl" scale="0.001 0.001 0.001"/>
+      </geometry>
+      <origin rpy="0 0 1.5708" />
+    </collision>
+    <inertial>
+        <mass value="0.01" />
+        <inertia ixx="0.001" ixy="0.0" ixz="0.0" iyy="0.001" iyz="0.0" izz="0.001" />
+    </inertial>
+    <visual>
+      <geometry>
+        <mesh filename="package://tr3_description/meshes/stl/tr-bs-b.stl" scale="0.001 0.001 0.001"/>
+      </geometry>
+      <material name="slate_gray">
+        <color rgba="0.2 0.2 0.2 1"/>
+      </material>
+      <origin rpy="0 0 1.5708" />
+    </visual>
+  </link>
+  <link name="link_b5">
+    <collision>
+      <geometry>
+        <mesh filename="package://tr3_description/meshes/stl/tr-bs-c.stl" scale="0.001 0.001 0.001"/>
+      </geometry>
+      <origin rpy="0 0 1.5708" />
+    </collision>
+    <inertial>
+        <mass value="0.01" />
+        <inertia ixx="0.001" ixy="0.0" ixz="0.0" iyy="0.001" iyz="0.0" izz="0.001" />
+    </inertial>
+    <visual>
+      <geometry>
+        <mesh filename="package://tr3_description/meshes/stl/tr-bs-c.stl" scale="0.001 0.001 0.001"/>
+      </geometry>
+      <material name="slate_gray">
+        <color rgba="0.2 0.2 0.2 1"/>
+      </material>
+      <origin rpy="0 0 1.5708" />
+    </visual>
+  </link>
+  <joint name="b2" type="continuous">
+    <parent link="base_link"/>
+    <child link="link_b2"/>
+    <origin xyz="-0.147 -0.39975 -0.09635" rpy="0 3.1415 -1.5708"/>
+    <axis xyz="0 0 1"/>
+    <dynamics damping="0.1" friction="0.1"/>
+  </joint>
+  <joint name="b3" type="continuous">
+    <parent link="link_b2"/>
+    <child link="link_b3"/>
+    <origin xyz="-0.0138 0 0.0390" rpy="1.5708 0 0"/>
+    <axis xyz="0 0 1"/>
+    <dynamics damping="0.1" friction="0.1"/>
+  </joint>
+  <joint name="b4" type="continuous">
+    <parent link="base_link"/>
+    <child link="link_b4"/>
+    <origin xyz="0.147 -0.39975 -0.09635" rpy="0 3.1415 -1.5708"/>
+    <axis xyz="0 0 1"/>
+    <dynamics damping="0.1" friction="0.1"/>
+  </joint>
+  <joint name="b5" type="continuous">
+    <parent link="link_b4"/>
+    <child link="link_b5"/>
+    <origin xyz="-0.0138 0 0.0390" rpy="1.5708 0 0"/>
+    <axis xyz="0 0 1"/>
+    <dynamics damping="0.1" friction="0.1"/>
+  </joint>
   <joint name="rplidar_joint" type="fixed">
     <axis xyz="0 0 1" />

Commit message: gazebo and server optimizations

File: tr3_description/urdf/base/base.gazebo.xacro (robot description, xacro)
@@ -1,25 +1,4 @@
 <?xml version="1.0"?>
 <robot xmlns:xacro="http://www.ros.org/wiki/xacro">
-	<gazebo reference="link_b0">
-		<material>Gazebo/DarkGrey</material>
-		<collision>
-      <surface>
-			  <contact>
-		      <ode>
-		        <kp>1e15</kp>
-		        <kd>1e13</kd>
-		      </ode>
-		    </contact>
-        <friction>
-          <ode>
-            <mu>100000.0</mu>
-            <mu2>100000.0</mu2>
-            <slip1>0.0</slip1>
-            <slip2>0.0</slip2>
-          </ode>
-        </friction>
-      </surface>
-		</collision>
-	</gazebo>
   <gazebo reference="laser">
     <sensor type="gpu_ray" name="head_rplidar_sensor">
@@ -56,6 +35,8 @@
 		<material>Gazebo/DarkGrey</material>
 	</gazebo>
-	<gazebo reference="link_b1">
+	<gazebo reference="link_b0">
 		<material>Gazebo/DarkGrey</material>
+    <mu1 value="100000.0"/>
+    <mu2 value="100000.0"/>
 		<collision>
       <surface>
@@ -77,15 +58,62 @@
 		</collision>
 	</gazebo>
-	<gazebo reference="link_b2">
+	<gazebo reference="link_b1">
 		<material>Gazebo/DarkGrey</material>
+    <mu1 value="100000.0"/>
+    <mu2 value="100000.0"/>
+		<collision>
+      <surface>
+			  <contact>
+		      <ode>
+		        <kp>1e15</kp>
+		        <kd>1e13</kd>
+		      </ode>
+		    </contact>
+        <friction>
+          <ode>
+            <mu>100000.0</mu>
+            <mu2>100000.0</mu2>
+            <slip1>0.0</slip1>
+            <slip2>0.0</slip2>
+          </ode>
+        </friction>
+      </surface>
+		</collision>
 	</gazebo>
-	<gazebo reference="link_b3">
-		<material>Gazebo/DarkGrey</material>
-	</gazebo>
-	<gazebo reference="link_b4">
-		<material>Gazebo/DarkGrey</material>
-	</gazebo>
-	<gazebo reference="link_b5">
-		<material>Gazebo/DarkGrey</material>
-	</gazebo>
+  <gazebo reference="link_b2">
+    <mu1 value="0.1"/>
+    <mu2 value="0.1"/>
+    <kp value="10000000.0"/>
+    <kd value="1.0"/>
+    <fdir1 value="1 0 0"/>
+  	<material>Gazebo/DarkGrey</material>
+    <turnGravityOff>false</turnGravityOff>
+  </gazebo>
+  <gazebo reference="link_b3">
+    <mu1 value="0.1"/>
+    <mu2 value="0.1"/>
+    <kp value="10000000.0"/>
+    <kd value="1.0"/>
+    <fdir1 value="1 0 0"/>
+  	<material>Gazebo/DarkGrey</material>
+    <turnGravityOff>false</turnGravityOff>
+  </gazebo>
+  <gazebo reference="link_b4">
+    <mu1 value="0.1"/>
+    <mu2 value="0.1"/>
+    <kp value="10000000.0"/>
+    <kd value="1.0"/>
+    <fdir1 value="1 0 0"/>
+  	<material>Gazebo/DarkGrey</material>
+    <turnGravityOff>false</turnGravityOff>
+  </gazebo>
+  <gazebo reference="link_b5">
+    <mu1 value="0.1"/>
+    <mu2 value="0.1"/>
+    <kp value="10000000.0"/>
+    <kd value="1.0"/>
+    <fdir1 value="1 0 0"/>
+  	<material>Gazebo/DarkGrey</material>
+    <turnGravityOff>false</turnGravityOff>
+  </gazebo>
 </robot>

File: tr3_description/urdf/base/base.urdf.xacro (robot description, xacro)
@@ -9,7 +9,7 @@
 			<child link="link_${name}"/>
 			<xacro:insert_block name="axis" />
-			<limit effort="100.0" velocity="8.8"/>
+			<limit effort="100.0" velocity="0.5"/>
 			<xacro:insert_block name="origin" />
-    	<dynamics damping="0.001" friction="0.001"/>
+    	<dynamics damping="0.001" friction="0.1"/>
 		</joint>
 		<link name="link_${name}">

File: tr3_description/urdf/head/head.gazebo.xacro (robot description, xacro)
@@ -17,5 +17,5 @@
 				<clip>
 					<near>0.6</near>
-					<far>8.0</far>
+					<far>25.0</far>
 				</clip>
 			</camera>
