Commit message: configuring for real hardware

File: tr3_description/urdf/base/base.urdf.xacro (robot description, xacro)
@@ -172,5 +172,5 @@
   <joint name="rplidar_joint" type="fixed">
     <axis xyz="0 0 1" />
-    <origin xyz="0.11 0 0" rpy="0 0 -1.5708" />
+    <origin xyz="0.11 0 0" rpy="0 0 3.1415" />
     <parent link="base_link" />
     <child link="laser" />

Commit message: base urdf changes, updating TR_OS apps

File: tr3_description/urdf/base/base.urdf.xacro (robot description, xacro)
@@ -186,3 +186,10 @@
 		<origin rpy="0 0 3.1415" xyz="0 -0.3281 0"/>
 	</xacro:tr3_wheel>
+	<!-- dummy link required in order to specify base_link inertia because MoveIt is insane -->
+  <link name="dummy_link">
+  </link>
+  <joint name="dummy_joint" type="fixed">
+     <parent link="dummy_link"/>
+     <child link="base_link"/>
+   </joint>
 </robot>
